File: dohikey.kicad_pcb (KiCad board)
At the start: 2 copper layers, 61.5 x 53.5 mm, 11 parts, among them J1 Conn_01x04_Pin, J2 DHT11, J3 Motor, J4 Barrel_Jack_Switch_Pin3Ring, Q1 PN2222A

Commit message: Add files via upload
Fixed LCD miswire. Data and Clock pins were swapped.
Connections:
- J1 pad 3: Net-(A1-A5) -> Net-(A1-A4)
- J1 pad 4: Net-(A1-A4) -> Net-(A1-A5)
Routing:
- net Net-(A1-A5): track 6.81 -> 10.5 mm
Changed lines of the file:
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@@
 			(layers "*.Cu" "*.Mask")
 			(remove_unused_layers no)
-			(net 18 "Net-(A1-A5)")
+			(net 2 "Net-(A1-A4)")
 			(pinfunction "Pin_3")
 			(pintype "passive")
@@
 			(layers "*.Cu" "*.Mask")
 			(remove_unused_layers no)
-			(net 2 "Net-(A1-A4)")
+			(net 18 "Net-(A1-A5)")
 			(pinfunction "Pin_4")
 			(pintype "passive")
@@
 	)
 	(segment
-		(start 78.6 49.6)
-		(end 74.38 49.6)
+		(start 78.6 48.6)
+		(end 73.38 48.6)
 		(width 0.2)
 		(layer "F.Cu")
@@
 	)
 	(segment
-		(start 74.38 49.6)
+		(start 73.38 48.6)
 		(end 73 48.22)
 		(width 0.2)
@@
 	)
 	(segment
-		(start 78.6 48.6)
-		(end 75.92 48.6)
+		(start 72.82295 49.6)
+		(end 71.899 48.67605)
 		(width 0.2)
 		(layer "F.Cu")
@@
 	)
 	(segment
-		(start 75.92 48.6)
+		(start 78.6 49.6)
+		(end 72.82295 49.6)
+		(width 0.2)
+		(layer "F.Cu")
+		(net 18)
+	)
+	(segment
+		(start 71.899 46.781)
 		(end 73 45.68)
 		(width 0.2)
 		(layer "F.Cu")
+		(net 18)
+	)
+	(segment
+		(start 71.899 48.67605)
+		(end 71.899 46.781)
+		(width 0.2)
+		(layer "F.Cu")
